File: pcb/io_modul.kicad_pcb (KiCad board)
At the start: 2 copper layers, 50 x 25 mm, 23 parts, among them IC1 ATMEGA8-AI, J1 USB, P1 ISP, P2 Comunication, P3 Input/Output, U1 MCP4725A0T, U2 MCP4725A0T, X1 16MHz

Commit message: PCB modified
Parts:
- added D4: LED, LEDs:LED-0805, F.Cu at (121.7, 84.5)
- added R7: 150, SMD_Packages:SM0603_Resistor, F.Cu at (124.7, 86.6)
- moved D1 3.84 mm to (129.6, 84.2)
- moved F1 1.14 mm to (133.5, 88.3)
- moved R4 0.85 mm to (135.8, 91.7)
Connections:
- J1 pad 5: GND -> (no net)
Routing:
- net Net-(F1-Pad2): track 7.11 -> 13.8 mm
- net GND: track 57.9 -> 63.2 mm, vias 10 -> 12
- net VDD: track 128.1 -> 124.6 mm
- net Net-(D4-Pad2): track 0.00 -> 3.03 mm
- net /D-: track 18.8 -> 17.9 mm
- net (no net): vias 2 -> 0
Other:
- board text added: "IOUSB v1.0 ravit :-D 28.7. 2014"
