File: pcb/io_modul.sch (KiCad schematic (older format))
At the start: 23 parts, among them IC1 ATMEGA8-AI, J1 USB, P1 ISP, P2 Comunication, P3 Input/Output, U1 MCP4725A0T, U2 MCP4725A0T, X1 16MHz

Commit message: PCB modified
Parts:
- added D4: LED, symbol LED
- added R7: 150, symbol R
Connections:
- net GND: now also D4.1 (A); no longer J1.5 (Shield_1)
- net at F1.2, J1.1 (Vbus): now also R7.1
- new net: D4.2 (K), R7.2
- no-connect marks 3 -> 4
Other:
- note removed: "D/A convertor"
- moved on the sheet: C4, D1, F1
Changed lines of the file:
@@
 	2650 6350 2600 6350
 Connection ~ 2600 6350
-Wire Wire Line
-	2600 6450 3400 6450
-Wire Wire Line
-	3400 6450 3400 6350
-Connection ~ 2600 6450
 $Comp
 L FUSE F1
 U 1 1 53D13B6C
-P 2400 6100
-F 0 "F1" H 2500 6150 40  0000 C CNN
-F 1 "500mA" H 2300 6050 40  0000 C CNN
-F 2 "" H 2400 6100 60  0000 C CNN
-F 3 "" H 2400 6100 60  0000 C CNN
-	1    2400 6100
+P 1650 6100
+F 0 "F1" H 1750 6150 40  0000 C CNN
+F 1 "500mA" H 1550 6050 40  0000 C CNN
+F 2 "" H 1650 6100 60  0000 C CNN
+F 3 "" H 1650 6100 60  0000 C CNN
+	1    1650 6100
 	1    0    0    -1
 $EndComp
@@
 L VDD #PWR020
 U 1 1 53D13B88
-P 1350 6050
-F 0 "#PWR020" H 1350 6150 30  0001 C CNN
-F 1 "VDD" H 1350 6160 30  0000 C CNN
-F 2 "" H 1350 6050 60  0000 C CNN
-F 3 "" H 1350 6050 60  0000 C CNN
-	1    1350 6050
-	1    0    0    -1
-$EndComp
-Wire Wire Line
-	1350 6050 1350 6200
+P 800 6050
+F 0 "#PWR020" H 800 6150 30  0001 C CNN
+F 1 "VDD" H 800 6160 30  0000 C CNN
+F 2 "" H 800 6050 60  0000 C CNN
+F 3 "" H 800 6050 60  0000 C CNN
+	1    800  6050
+	1    0    0    -1
+$EndComp
+Wire Wire Line
+	800  6050 800  6200
 $Comp
 L R R2
@@
 L CP1 C4
 U 1 1 53D14175
-P 1350 6400
-F 0 "C4" H 1400 6500 50  0000 L CNN
-F 1 "4u7" H 1400 6300 50  0000 L CNN
-F 2 "" H 1350 6400 60  0000 C CNN
-F 3 "" H 1350 6400 60  0000 C CNN
-	1    1350 6400
+P 800 6400
+F 0 "C4" H 850 6500 50  0000 L CNN
+F 1 "4u7" H 850 6300 50  0000 L CNN
+F 2 "" H 800 6400 60  0000 C CNN
+F 3 "" H 800 6400 60  0000 C CNN
+	1    800  6400
 	1    0    0    -1
 $EndComp
@@
 L GND #PWR022
 U 1 1 53D14187
-P 1350 6600
-F 0 "#PWR022" H 1350 6600 30  0001 C CNN
-F 1 "GND" H 1350 6530 30  0001 C CNN
-F 2 "" H 1350 6600 60  0000 C CNN
-F 3 "" H 1350 6600 60  0000 C CNN
-	1    1350 6600
+P 800 6600
+F 0 "#PWR022" H 800 6600 30  0001 C CNN
+F 1 "GND" H 800 6530 30  0001 C CNN
+F 2 "" H 800 6600 60  0000 C CNN
+F 3 "" H 800 6600 60  0000 C CNN
+	1    800  6600
 	1    0    0    -1
 $EndComp
@@
 L DIODESCH D1
 U 1 1 53D22FD1
-P 1800 6300
-F 0 "D1" H 1800 6400 40  0000 C CNN
-F 1 "5V transil" H 1800 6200 40  0000 C CNN
-F 2 "" H 1800 6300 60  0000 C CNN
-F 3 "" H 1800 6300 60  0000 C CNN
-	1    1800 6300
+P 1250 6300
+F 0 "D1" H 1250 6400 40  0000 C CNN
+F 1 "5V transil" H 1250 6200 40  0000 C CNN
+F 2 "" H 1250 6300 60  0000 C CNN
+F 3 "" H 1250 6300 60  0000 C CNN
+	1    1250 6300
 	0    -1   -1   0
 $EndComp
 Wire Wire Line
-	1350 6100 2150 6100
-Connection ~ 1800 6100
-Connection ~ 1350 6100
+	800  6100 1400 6100
+Connection ~ 1250 6100
+Connection ~ 800  6100
 $Comp
 L GND #PWR024
 U 1 1 53D23211
-P 1800 6500
-F 0 "#PWR024" H 1800 6500 30  0001 C CNN
-F 1 "GND" H 1800 6430 30  0001 C CNN
-F 2 "" H 1800 6500 60  0000 C CNN
-F 3 "" H 1800 6500 60  0000 C CNN
-	1    1800 6500
+P 1250 6500
+F 0 "#PWR024" H 1250 6500 30  0001 C CNN
+F 1 "GND" H 1250 6430 30  0001 C CNN
+F 2 "" H 1250 6500 60  0000 C CNN
+F 3 "" H 1250 6500 60  0000 C CNN
+	1    1250 6500
 	1    0    0    -1
 $EndComp
@@
 Wire Wire Line
 	9850 2150 10150 2150
-Wire Notes Line
-	4900 500  4900 7800
-Wire Notes Line
-	500  5000 11200 5000
-Wire Notes Line
-	8800 5000 8800 500
-Text Notes 5100 800  0    60   ~ 0
-D/A convertor
+$Comp
+L LED D4
+U 1 1 53D674BF
+P 2050 6800
+F 0 "D4" H 2050 6900 50  0000 C CNN
+F 1 "LED" H 2050 6700 50  0000 C CNN
+F 2 "" H 2050 6800 60  0000 C CNN
+F 3 "" H 2050 6800 60  0000 C CNN
+	1    2050 6800
+	0    -1   -1   0
+$EndComp
+Wire Wire Line
+	1900 6100 2650 6100
+Connection ~ 2050 6100
+$Comp
+L R R7
+U 1 1 53D67575
+P 2050 6350
+F 0 "R7" V 2130 6350 40  0000 C CNN
+F 1 "150" V 2057 6351 40  0000 C CNN
+F 2 "" V 1980 6350 30  0000 C CNN
+F 3 "" H 2050 6350 30  0000 C CNN
+	1    2050 6350
+	1    0    0    -1
+$EndComp
+$Comp
+L GND #PWR032
+U 1 1 53D67591
+P 2050 7000
+F 0 "#PWR032" H 2050 7000 30  0001 C CNN
+F 1 "GND" H 2050 6930 30  0001 C CNN
+F 2 "" H 2050 7000 60  0000 C CNN
+F 3 "" H 2050 7000 60  0000 C CNN
+	1    2050 7000
+	1    0    0    -1
+$EndComp
+NoConn ~ 3400 6350
 $EndSCHEMATC
